File: pcb/smart-lcc/smart-lcc.sch (KiCad schematic (older format))
At the start: 30 parts, among them J1 280372-1, J2 Aux connector, J3 Conn_01x24 (mirrored), SW1 SW_Push, SW2 SW_Push, U1 ABX00027, U2 LPV358, U3 LPV358

Commit message: WIP
Parts:
- removed D10, D5, D7, D8: D_Small, Diode_SMD:D_SOD-123, symbol Device:D_Small
- removed U2, U3: LPV358, Package_SO:VSSOP-8_3.0x3.0mm_P0.65mm, symbol Amplifier_Operational:LM358
- added D6, D7: D_Zener_Small, Diode_SMD:D_SOD-123, symbol Device:D_Zener_Small
- added H1, H2, H3, H4: MountingHole, MountingHole:MountingHole_2.7mm, symbol Mechanical:MountingHole
- added Q1, Q2, Q3, Q4: 2N7002, Package_TO_SOT_SMD:SOT-23, symbol Transistor_FET:2N7002
- added R3, R4, R5: 220R, Resistor_SMD:R_0402_1005Metric, symbol Device:R_Small
- C1: footprint Capacitor_SMD:C_0603_1608Metric -> Capacitor_SMD:C_0805_2012Metric; Comment Per display data sheet reference design -> Per display data sheet reference design, part is 50V; JLCPCB Basic N -> Y; LCSC C57895 -> C49217
- C2: footprint Capacitor_SMD:C_0805_2012Metric -> Capacitor_SMD:C_1206_3216Metric; Comment Per display data sheet reference design -> Per display data sheet reference design, part is 50V; JLCPCB Basic N -> Y; LCSC C98195 -> C29823
- J3: value Conn_01x24 (mirrored) -> Conn_01x24; footprint Connector_FFC-FPC:Hirose_FH12-24S-0.5SH_1x24-1MP_P0.50mm_Horizontal -> FH34SRJ-24S-0.5SH_50:FH34SRJ24S05SH50
- R1: symbol Device:R -> Device:R_Small; JLCPCB Basic N -> Y; LCSC C138019 -> C25879
- R2: symbol Device:R -> Device:R_Small; JLCPCB Basic N -> Y; LCSC C137993 -> C25890
- renumbered D3 to D2, D4 to D3, D2 to D4, D6 to D5, D9 to D8, R3 to R10, R4 to R6, R6 to R7, R7 to R8, R5 to R9, SW2 to SW1, SW1 to SW2
Connections:
- net +12V: now also J3.23 (Pin_23); no longer J3.2 (Pin_2)
- net +3V3: now also R6.2, R7.2, R8.2, R9.2
- net 3V3_OLED: now also J3.5 (Pin_5); no longer J3.20 (Pin_20)
- net GND: now also J3.11 (Pin_11), J3.12 (Pin_12), J3.16 (Pin_16), J3.17 (Pin_17), J3.2 (Pin_2), J3.20 (Pin_20), J3.3 (Pin_3), D6.2 (A), D7.2 (A), Q1.2 (S), Q2.2 (S), Q3.2 (S), Q4.2 (S); no longer D1.1 (K), D2.1 (K), D3.1 (K), D4.1 (K), J3.13 (Pin_13), J3.14 (Pin_14), J3.22 (Pin_22), J3.23 (Pin_23), J3.5 (Pin_5), J3.8 (Pin_8), J3.9 (Pin_9)
- net RX_FROM_AUX: now also Q3.1 (G), R5.2
- net RX_FROM_CONTROL_BOARD_3V3: now also D5.1 (K), U1.17 (RX), Q1.1 (G)
- net SSD1309_CS: now also J3.8 (Pin_8); no longer J3.17 (Pin_17)
- net SSD1309_DC: now also J3.10 (Pin_10); no longer J3.15 (Pin_15)
- net SSD1309_MOSI: now also J3.14 (Pin_14); no longer J3.11 (Pin_11)
- net SSD1309_RES: now also J3.9 (Pin_9); no longer J3.16 (Pin_16)
- net SSD1309_SCLK: now also J3.13 (Pin_13); no longer J3.12 (Pin_12)
- net TX_TO_AUX: now also Q4.1 (G), R4.1
- net TX_TO_CONTROL_BOARD: now also Q2.1 (G), R3.2
- net at U1.16 (TX): now also D6.1 (K), R3.1
- net at U1.26 (D8): now also D7.1 (K), R4.2
- net at D8.1 (K), U1.27 (D9/PWM): now also R5.1
- net at R10.2: now also J3.21 (Pin_21); no longer J3.4 (Pin_4)
- net at C1.1: now also J3.22 (Pin_22); no longer J3.3 (Pin_3)
- new net: D1.1 (K), Q1.3 (D)
- new net: D2.1 (K), Q2.3 (D)
- new net: D4.1 (K), Q4.3 (D)
- new net: D3.1 (K), Q3.3 (D)
- no-connect marks 12 -> 16
Other:
- moved on the sheet: C1, C2, C3, D1, D2, D3, D4, D5, D8, J3, R1, R10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

Commit message: Rev B as sent to manufacturing
Parts:
- J3: LCSC C506794 -> C324726
Changed lines of the file:
@@
 F 3 "~" H 5500 2400 50  0001 C CNN
 F 4 "N" H 5500 2400 50  0001 C CNN "JLCPCB Basic"
-F 5 "C506794" H 5500 2400 50  0001 C CNN "LCSC"
+F 5 "C324726" H 5500 2400 50  0001 C CNN "LCSC"
 	1    5500 2400
 	1    0    0    1
